File: openLRSngRX32.sch (EAGLE design)
At the start: 19 parts, among them IC1 STM32F10XCXT6, IC2 REG1117

Commit message: - remove project - working onwards...
Parts:
- added C1, C10, C11, C2, C3, C4, C5, C6, C7, C8, C9: (no value), SparkFun-Capacitors:CAP0805
- added JP4: (no value), SparkFun-Connectors:M04PTH
- added JP5, JP6: (no value), SparkFun-Connectors:M06SIP
- added JP7, JP8: (no value), SparkFun-Connectors:M02PTH
- added R13, R14, R15, R16: (no value), SparkFun-Resistors:RESISTOR0805-RES
- added U1: MPU-6000QFN-24, SparkFun-Sensors:MPU-6000QFN-24
- added Y1: (no value), crystal_3225:CRYSTAL3.2X2.5
Connections:
- new net BOOT0: IC1RESET.BOOT0, JP7.2, R15.2
- new net DTR: JP5.6
- new net MPUINT: U1.INT
- new net N$14: C1.2, U1.REGOUT
- new net N$15: C2.2, U1.CPOUT
- new net N$16: C4.1, IC1PORTD/OSC.PD0/OSC<=, Y1.2
- new net N$17: C3.1, IC1PORTD/OSC.PD1/OSC=>, Y1.1
- new net N$29: JP5.2
- new net N$35: JP6.3
- new net PPM: IC1PORTA_H.PA8, JP6.6
- new net RESET: C11.1, IC1RESET.NRST, JP8.1, R16.1
- new net RX: IC1PORTA_H.PA10, JP5.4
- new net SCL: IC1PORTB_H.PB10, JP4.3, R13.1, U1.SCL/SCLK
- new net SDA: IC1PORTB_H.PB11, JP4.2, R14.1, U1.SDA/SDI
- new net TX: IC1PORTA_H.PA9, JP5.5
- net 3V3: now also C10.1, C5.1, C6.1, C7.1, C8.1, C9.1, JP4.4, JP5.3, JP7.1, R13.2, R14.2, R16.2, U1.CS, U1.VDD
- net GND: now also C1.1, C10.2, C11.2, C2.1, C3.2, C4.2, C5.2, C6.2, C7.2, C8.2, C9.2, JP4.1, JP5.1, JP6.1, JP6.4, JP8.2, R15.1, U1.AD0/SDO, U1.CLKIN, U1.FSYNC, U1.GND, Y1.GND
- net VCC: now also JP6.2, JP6.5

Commit message: some more caps
Parts:
- added C12, C13: (no value), SparkFun-Capacitors:CAP0805
- added C14: 47uF, SparkFun-Capacitors:47UF-TANT
Connections:
- net 3V3: now also C14.+
- net GND: now also C12.2, C13.2, C14.-
- net VCC: now also C12.1, C13.1
Changed lines of the file:
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@@
 <part name="JP8" library="SparkFun-Connectors" deviceset="M02" device="PTH"/>
 <part name="GND16" library="supply1" deviceset="GND" device=""/>
+<part name="C12" library="SparkFun-Capacitors" deviceset="CAP" device="0805"/>
+<part name="C13" library="SparkFun-Capacitors" deviceset="CAP" device="0805"/>
+<part name="C14" library="SparkFun-Capacitors" deviceset="47UF-TANT" device="" value="47uF"/>
 </parts>
 <sheets>
@@
 <instance part="JP8" gate="G$1" x="119.38" y="-20.32" rot="R180"/>
 <instance part="GND16" gate="1" x="106.68" y="-25.4"/>
+<instance part="C12" gate="G$1" x="-22.86" y="30.48"/>
+<instance part="C13" gate="G$1" x="-27.94" y="30.48"/>
+<instance part="C14" gate="G$1" x="2.54" y="33.02"/>
 </instances>
 <busses>
@@
 <pinref part="GND2" gate="1" pin="GND"/>
 <wire x1="-10.16" y1="22.86" x2="-10.16" y2="20.32" width="0.1524" layer="91"/>
+<pinref part="C13" gate="G$1" pin="2"/>
+<wire x1="-10.16" y1="22.86" x2="-22.86" y2="22.86" width="0.1524" layer="91"/>
+<wire x1="-22.86" y1="22.86" x2="-27.94" y2="22.86" width="0.1524" layer="91"/>
+<wire x1="-27.94" y1="22.86" x2="-27.94" y2="27.94" width="0.1524" layer="91"/>
+<pinref part="C12" gate="G$1" pin="2"/>
+<wire x1="-22.86" y1="27.94" x2="-22.86" y2="22.86" width="0.1524" layer="91"/>
+<junction x="-22.86" y="22.86"/>
+<junction x="-10.16" y="22.86"/>
+<pinref part="C14" gate="G$1" pin="-"/>
+<wire x1="-10.16" y1="22.86" x2="2.54" y2="22.86" width="0.1524" layer="91"/>
+<wire x1="2.54" y1="22.86" x2="2.54" y2="27.94" width="0.1524" layer="91"/>
 </segment>
 <segment>
@@
 <pinref part="IC2" gate="G$1" pin="VIN"/>
 <wire x1="-22.86" y1="40.64" x2="-22.86" y2="35.56" width="0.1524" layer="91"/>
+<pinref part="C12" gate="G$1" pin="1"/>
+<junction x="-22.86" y="35.56"/>
+<pinref part="C13" gate="G$1" pin="1"/>
+<wire x1="-27.94" y1="35.56" x2="-22.86" y2="35.56" width="0.1524" layer="91"/>
 </segment>
 <segment>
@@
 <wire x1="2.54" y1="35.56" x2="5.08" y2="35.56" width="0.1524" layer="91"/>
 <label x="5.08" y="35.56" size="1.778" layer="95"/>
-</segment>
-<segment>
+<pinref part="C14" gate="G$1" pin="+"/>
+<junction x="2.54" y="35.56"/>
+</segment>
+<segment>

Commit message: board
Parts:
- added J$1, J$2: SMA_EDGE, SparkFun-Connectors:SMA_EDGE
- added JP9: (no value), SparkFun-Connectors:M03PTH
- added R17: (no value), SparkFun-Resistors:RESISTOR0805-RES
- JP6: device SparkFun-Connectors:M06SIP -> SparkFun-Connectors:M03PTH
Connections:
- removed net N$35: JP6.3
- new net N$13: J$2.SIGNAL, U$2.ANT
- new net N$18: J$1.SIGNAL, U$1.ANT
- new net N$19: U$2.GPIO0, U$2.TXANT
- new net N$20: U$2.GPIO1, U$2.RXANT
- new net N$23: U$1.GPIO0, U$1.TXANT
- new net N$24: U$1.GPIO1, U$1.RXANT
- new net N$25: JP6.3, R17.1
- net GND: now also J$1.GND@0, J$1.GND@1, J$1.GND@2, J$1.GND@3, J$2.GND@0, J$2.GND@1, J$2.GND@2, J$2.GND@3; no longer JP6.4
- net PPM: now also R17.2; no longer JP6.6
- net VCC: no longer JP6.5
Changed lines of the file:
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@@
 <part name="JP4" library="SparkFun-Connectors" deviceset="M04" device="PTH"/>
 <part name="JP5" library="SparkFun-Connectors" deviceset="M06" device="SIP"/>
-<part name="JP6" library="SparkFun-Connectors" deviceset="M06" device="SIP"/>
 <part name="P+3" library="supply1" deviceset="VCC" device=""/>
 <part name="GND11" library="supply1" deviceset="GND" device=""/>
@@
 <part name="C13" library="SparkFun-Capacitors" deviceset="CAP" device="0805"/>
 <part name="C14" library="SparkFun-Capacitors" deviceset="47UF-TANT" device="" value="47uF"/>
+<part name="J$1" library="SparkFun-Connectors" deviceset="SMA_EDGE" device=""/>
+<part name="J$2" library="SparkFun-Connectors" deviceset="SMA_EDGE" device=""/>
+<part name="GND17" library="supply1" deviceset="GND" device=""/>
+<part name="JP6" library="SparkFun-Connectors" deviceset="M03" device="PTH"/>
+<part name="JP9" library="SparkFun-Connectors" deviceset="M03" device="PTH"/>
+<part name="R17" library="SparkFun-Resistors" deviceset="RESISTOR" device="0805-RES"/>
 </parts>
 <sheets>
@@
 <instance part="JP4" gate="G$1" x="-66.04" y="88.9"/>
 <instance part="JP5" gate="G$1" x="-66.04" y="68.58"/>
-<instance part="JP6" gate="G$1" x="-43.18" y="68.58"/>
-<instance part="P+3" gate="VCC" x="-35.56" y="83.82"/>
-<instance part="GND11" gate="1" x="-33.02" y="55.88"/>
+<instance part="P+3" gate="VCC" x="-30.48" y="83.82"/>
+<instance part="GND11" gate="1" x="-33.02" y="48.26"/>
 <instance part="C11" gate="G$1" x="88.9" y="5.08"/>
 <instance part="R15" gate="G$1" x="71.12" y="0" rot="R90"/>
@@
 <instance part="C13" gate="G$1" x="-27.94" y="30.48"/>
 <instance part="C14" gate="G$1" x="2.54" y="33.02"/>
+<instance part="J$1" gate="1" x="147.32" y="81.28" rot="R180"/>
+<instance part="J$2" gate="1" x="147.32" y="40.64" rot="R180"/>
+<instance part="GND17" gate="1" x="157.48" y="83.82"/>
+<instance part="JP6" gate="G$1" x="-45.72" y="73.66"/>
+<instance part="JP9" gate="G$1" x="-45.72" y="58.42"/>
+<instance part="R17" gate="G$1" x="-35.56" y="81.28" rot="R90"/>
 </instances>
 <busses>
@@
 </segment>
 <segment>
-<pinref part="JP6" gate="G$1" pin="4"/>
 <wire x1="-38.1" y1="71.12" x2="-33.02" y2="71.12" width="0.1524" layer="91"/>
-<wire x1="-33.02" y1="71.12" x2="-33.02" y2="63.5" width="0.1524" layer="91"/>
+<wire x1="-33.02" y1="71.12" x2="-33.02" y2="55.88" width="0.1524" layer="91"/>
+<wire x1="-33.02" y1="55.88" x2="-38.1" y2="55.88" width="0.1524" layer="91"/>
+<pinref part="GND11" gate="1" pin="GND"/>
+<wire x1="-33.02" y1="50.8" x2="-33.02" y2="55.88" width="0.1524" layer="91"/>
+<junction x="-33.02" y="55.88"/>
 <pinref part="JP6" gate="G$1" pin="1"/>
-<wire x1="-33.02" y1="63.5" x2="-38.1" y2="63.5" width="0.1524" layer="91"/>
-<pinref part="GND11" gate="1" pin="GND"/>
-<wire x1="-33.02" y1="58.42" x2="-33.02" y2="63.5" width="0.1524" layer="91"/>
-<junction x="-33.02" y="63.5"/>
 </segment>
 <segment>
@@
 <pinref part="GND16" gate="1" pin="GND"/>
 <wire x1="106.68" y1="-22.86" x2="111.76" y2="-22.86" width="0.1524" layer="91"/>
+</segment>
+<segment>
+<pinref part="J$2" gate="1" pin="GND@0"/>
+<pinref part="J$1" gate="1" pin="GND@3"/>
+<wire x1="149.86" y1="45.72" x2="149.86" y2="48.26" width="0.1524" layer="91"/>
+<wire x1="149.86" y1="48.26" x2="149.86" y2="50.8" width="0.1524" layer="91"/>
+<wire x1="149.86" y1="50.8" x2="149.86" y2="53.34" width="0.1524" layer="91"/>
+<wire x1="149.86" y1="53.34" x2="149.86" y2="86.36" width="0.1524" layer="91"/>
+<wire x1="149.86" y1="86.36" x2="149.86" y2="88.9" width="0.1524" layer="91"/>
+<wire x1="149.86" y1="88.9" x2="149.86" y2="91.44" width="0.1524" layer="91"/>
+<wire x1="149.86" y1="91.44" x2="149.86" y2="93.98" width="0.1524" layer="91"/>
+<wire x1="149.86" y1="93.98" x2="157.48" y2="93.98" width="0.1524" layer="91"/>
+<wire x1="157.48" y1="93.98" x2="157.48" y2="86.36" width="0.1524" layer="91"/>
+<pinref part="GND17" gate="1" pin="GND"/>
+<pinref part="J$1" gate="1" pin="GND@0"/>
+<junction x="149.86" y="86.36"/>
+<pinref part="J$1" gate="1" pin="GND@1"/>
+<junction x="149.86" y="88.9"/>
+<pinref part="J$1" gate="1" pin="GND@2"/>
+<junction x="149.86" y="91.44"/>
+<junction x="149.86" y="93.98"/>
+<pinref part="J$2" gate="1" pin="GND@1"/>
+<junction x="149.86" y="48.26"/>
+<pinref part="J$2" gate="1" pin="GND@2"/>
+<junction x="149.86" y="50.8"/>
+<pinref part="J$2" gate="1" pin="GND@3"/>
+<junction x="149.86" y="53.34"/>
 </segment>
 </net>
@@
 </segment>
 <segment>
-<pinref part="JP6" gate="G$1" pin="5"/>
-<wire x1="-38.1" y1="73.66" x2="-35.56" y2="73.66" width="0.1524" layer="91"/>
+<wire x1="-38.1" y1="73.66" x2="-30.48" y2="73.66" width="0.1524" layer="91"/>
+<wire x1="-30.48" y1="73.66" x2="-30.48" y2="81.28" width="0.1524" layer="91"/>
+<pinref part="P+3" gate="VCC" pin="VCC"/>
 <pinref part="JP6" gate="G$1" pin="2"/>
-<wire x1="-38.1" y1="66.04" x2="-35.56" y2="66.04" width="0.1524" layer="91"/>
-<wire x1="-35.56" y1="73.66" x2="-35.56" y2="66.04" width="0.1524" layer="91"/>
-<wire x1="-35.56" y1="73.66" x2="-35.56" y2="81.28" width="0.1524" layer="91"/>
-<pinref part="P+3" gate="VCC" pin="VCC"/>
-<junction x="-35.56" y="73.66"/>
 </segment>
 </net>
@@
 <net name="PPM" class="0">
 <segment>
-<pinref part="JP6" gate="G$1" pin="6"/>
-<wire x1="-38.1" y1="76.2" x2="-30.48" y2="76.2" width="0.1524" layer="91"/>
-<label x="-33.02" y="76.2" size="1.778" layer="95"/>
-</segment>
-<segment>
 <pinref part="IC1" gate="PORTA_H" pin="PA8"/>
 <wire x1="48.26" y1="68.58" x2="45.72" y2="68.58" width="0.1524" layer="91"/>
 <label x="40.64" y="68.58" size="1.778" layer="95"/>
 </segment>
-</net>
-<net name="N$35" class="0">
-<segment>
-<pinref part="JP6" gate="G$1" pin="3"/>
-<wire x1="-38.1" y1="68.58" x2="-30.48" y2="68.58" width="0.1524" layer="91"/>
+<segment>
+<pinref part="R17" gate="G$1" pin="2"/>
+<wire x1="-35.56" y1="86.36" x2="-35.56" y2="88.9" width="0.1524" layer="91"/>
 </segment>
 </net>
@@
 </segment>
 </net>
+<net name="N$13" class="0">
+<segment>
+<pinref part="U$2" gate="G$1" pin="ANT"/>
+<pinref part="J$2" gate="1" pin="SIGNAL"/>
+<wire x1="134.62" y1="40.64" x2="142.24" y2="40.64" width="0.1524" layer="91"/>
+</segment>
+</net>
+<net name="N$18" class="0">
+<segment>
+<pinref part="U$1" gate="G$1" pin="ANT"/>
+<pinref part="J$1" gate="1" pin="SIGNAL"/>
+<wire x1="134.62" y1="81.28" x2="142.24" y2="81.28" width="0.1524" layer="91"/>
+</segment>
+</net>
+<net name="N$19" class="0">
+<segment>
+<pinref part="U$2" gate="G$1" pin="TXANT"/>
+<wire x1="134.62" y1="22.86" x2="137.16" y2="22.86" width="0.1524" layer="91"/>
+<wire x1="137.16" y1="22.86" x2="137.16" y2="17.78" width="0.1524" layer="91"/>
+<pinref part="U$2" gate="G$1" pin="GPIO0"/>
+<wire x1="137.16" y1="17.78" x2="134.62" y2="17.78" width="0.1524" layer="91"/>
+</segment>
+</net>
+<net name="N$20" class="0">
+<segment>
+<pinref part="U$2" gate="G$1" pin="GPIO1"/>
+<wire x1="134.62" y1="15.24" x2="139.7" y2="15.24" width="0.1524" layer="91"/>
+<wire x1="139.7" y1="15.24" x2="139.7" y2="25.4" width="0.1524" layer="91"/>
+<pinref part="U$2" gate="G$1" pin="RXANT"/>
+<wire x1="139.7" y1="25.4" x2="134.62" y2="25.4" width="0.1524" layer="91"/>
+</segment>
+</net>
+<net name="N$23" class="0">
+<segment>
+<pinref part="U$1" gate="G$1" pin="TXANT"/>
+<wire x1="134.62" y1="63.5" x2="137.16" y2="63.5" width="0.1524" layer="91"/>
+<wire x1="137.16" y1="63.5" x2="137.16" y2="58.42" width="0.1524" layer="91"/>
+<pinref part="U$1" gate="G$1" pin="GPIO0"/>
+<wire x1="137.16" y1="58.42" x2="134.62" y2="58.42" width="0.1524" layer="91"/>
+</segment>
+</net>
+<net name="N$24" class="0">
+<segment>
+<pinref part="U$1" gate="G$1" pin="GPIO1"/>
+<wire x1="134.62" y1="55.88" x2="139.7" y2="55.88" width="0.1524" layer="91"/>
+<wire x1="139.7" y1="55.88" x2="139.7" y2="66.04" width="0.1524" layer="91"/>
+<pinref part="U$1" gate="G$1" pin="RXANT"/>
+<wire x1="139.7" y1="66.04" x2="134.62" y2="66.04" width="0.1524" layer="91"/>
+</segment>
+</net>
+<net name="N$25" class="0">
+<segment>
+<pinref part="JP6" gate="G$1" pin="3"/>
+<pinref part="R17" gate="G$1" pin="1"/>
+<wire x1="-35.56" y1="76.2" x2="-38.1" y2="76.2" width="0.1524" layer="91"/>
+</segment>
+</net>

Commit message: pcb
Parts:
- added JP10: (no value), SparkFun-Connectors:M03PTH
Connections:
- new net AIN4: IC1PORTA_L.PA4, JP9.3
- new net AIN5: IC1PORTA_L.PA5, JP10.3
- net 3V3: now also JP10.2, JP9.2
- net GND: now also JP10.1, JP9.1
Other:
- moved on the sheet: JP9
Changed lines of the file:
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@@
 <part name="GND17" library="supply1" deviceset="GND" device=""/>
 <part name="JP6" library="SparkFun-Connectors" deviceset="M03" device="PTH"/>
+<part name="R17" library="SparkFun-Resistors" deviceset="RESISTOR" device="0805-RES"/>
 <part name="JP9" library="SparkFun-Connectors" deviceset="M03" device="PTH"/>
-<part name="R17" library="SparkFun-Resistors" deviceset="RESISTOR" device="0805-RES"/>
+<part name="JP10" library="SparkFun-Connectors" deviceset="M03" device="PTH"/>
 </parts>
 <sheets>
@@
 <instance part="JP5" gate="G$1" x="-66.04" y="68.58"/>
 <instance part="P+3" gate="VCC" x="-30.48" y="83.82"/>
-<instance part="GND11" gate="1" x="-33.02" y="48.26"/>
+<instance part="GND11" gate="1" x="-33.02" y="38.1"/>
 <instance part="C11" gate="G$1" x="88.9" y="5.08"/>
 <instance part="R15" gate="G$1" x="71.12" y="0" rot="R90"/>
@@
 <instance part="GND17" gate="1" x="157.48" y="83.82"/>
 <instance part="JP6" gate="G$1" x="-45.72" y="73.66"/>
-<instance part="JP9" gate="G$1" x="-45.72" y="58.42"/>
 <instance part="R17" gate="G$1" x="-35.56" y="81.28" rot="R90"/>
+<instance part="JP9" gate="G$1" x="-45.72" y="60.96"/>
+<instance part="JP10" gate="G$1" x="-45.72" y="48.26"/>
 </instances>
 <busses>
@@
 <segment>
 <wire x1="-38.1" y1="71.12" x2="-33.02" y2="71.12" width="0.1524" layer="91"/>
-<wire x1="-33.02" y1="71.12" x2="-33.02" y2="55.88" width="0.1524" layer="91"/>
-<wire x1="-33.02" y1="55.88" x2="-38.1" y2="55.88" width="0.1524" layer="91"/>
+<wire x1="-33.02" y1="71.12" x2="-33.02" y2="58.42" width="0.1524" layer="91"/>
 <pinref part="GND11" gate="1" pin="GND"/>
-<wire x1="-33.02" y1="50.8" x2="-33.02" y2="55.88" width="0.1524" layer="91"/>
-<junction x="-33.02" y="55.88"/>
 <pinref part="JP6" gate="G$1" pin="1"/>
+<pinref part="JP10" gate="G$1" pin="1"/>
+<wire x1="-33.02" y1="58.42" x2="-33.02" y2="45.72" width="0.1524" layer="91"/>
+<wire x1="-33.02" y1="45.72" x2="-33.02" y2="40.64" width="0.1524" layer="91"/>
+<wire x1="-33.02" y1="45.72" x2="-38.1" y2="45.72" width="0.1524" layer="91"/>
+<pinref part="JP9" gate="G$1" pin="1"/>
+<wire x1="-33.02" y1="58.42" x2="-38.1" y2="58.42" width="0.1524" layer="91"/>
+<junction x="-33.02" y="45.72"/>
+<junction x="-33.02" y="58.42"/>
 </segment>
 <segment>
@@
 <label x="101.6" y="-5.08" size="1.778" layer="95"/>
 </segment>
+<segment>
+<pinref part="JP9" gate="G$1" pin="2"/>
+<wire x1="-38.1" y1="60.96" x2="-30.48" y2="60.96" width="0.1524" layer="91"/>
+<wire x1="-30.48" y1="60.96" x2="-30.48" y2="48.26" width="0.1524" layer="91"/>
+<pinref part="JP10" gate="G$1" pin="2"/>
+<wire x1="-30.48" y1="48.26" x2="-38.1" y2="48.26" width="0.1524" layer="91"/>
+<wire x1="-30.48" y1="48.26" x2="-25.4" y2="48.26" width="0.1524" layer="91"/>
+<wire x1="-25.4" y1="48.26" x2="-25.4" y2="50.8" width="0.1524" layer="91"/>
+<label x="-25.4" y="50.8" size="1.778" layer="95"/>
+</segment>
 </net>
 <net name="N$1" class="0">
@@
 <pinref part="R17" gate="G$1" pin="2"/>
 <wire x1="-35.56" y1="86.36" x2="-35.56" y2="88.9" width="0.1524" layer="91"/>
+<label x="-35.56" y="88.9" size="1.778" layer="95"/>
 </segment>
 </net>
@@
 </segment>
 </net>
+<net name="AIN5" class="0">
+<segment>
+<wire x1="-38.1" y1="50.8" x2="-35.56" y2="50.8" width="0.1524" layer="91"/>
+<label x="-35.56" y="50.8" size="1.778" layer="95"/>
+<pinref part="JP10" gate="G$1" pin="3"/>
+</segment>
+<segment>
+<pinref part="IC1" gate="PORTA_L" pin="PA5"/>
+<wire x1="48.26" y1="81.28" x2="45.72" y2="81.28" width="0.1524" layer="91"/>
+<label x="40.64" y="81.28" size="1.778" layer="95"/>
+</segment>
+</net>
+<net name="AIN4" class="0">
+<segment>
+<wire x1="-38.1" y1="63.5" x2="-35.56" y2="63.5" width="0.1524" layer="91"/>
+<label x="-35.56" y="63.5" size="1.778" layer="95"/>
+<pinref part="JP9" gate="G$1" pin="3"/>
+</segment>
+<segment>
+<pinref part="IC1" gate="PORTA_L" pin="PA4"/>
+<wire x1="48.26" y1="83.82" x2="45.72" y2="83.82" width="0.1524" layer="91"/>
+<label x="40.64" y="83.82" size="1.778" layer="95"/>
+</segment>
+</net>

Commit message: updates
Parts:
- added C15: (no value), SparkFun-Capacitors:CAP0805
Connections:
- net 3V3: now also C15.1
- net GND: now also C15.2
- net PWM10: now also IC1PORTB_H.PB8; no longer IC1PORTB_L.PB7
- net PWM11: now also IC1PORTB_L.PB7; no longer IC1PORTB_H.PB8
- net PWM12: now also IC1PORTB_L.PB6; no longer IC1PORTB_H.PB9
- net PWM9: now also IC1PORTB_H.PB9; no longer IC1PORTB_L.PB6
Changed lines of the file:
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@@
 <part name="JP9" library="SparkFun-Connectors" deviceset="M03" device="PTH"/>
 <part name="JP10" library="SparkFun-Connectors" deviceset="M03" device="PTH"/>
+<part name="C15" library="SparkFun-Capacitors" deviceset="CAP" device="0805"/>
 </parts>
 <sheets>
@@
 <instance part="JP9" gate="G$1" x="-45.72" y="60.96"/>
 <instance part="JP10" gate="G$1" x="-45.72" y="48.26"/>
+<instance part="C15" gate="G$1" x="-43.18" y="33.02"/>
 </instances>
 <busses>
@@
 <junction x="-63.5" y="30.48"/>
 <junction x="-68.58" y="30.48"/>
+<pinref part="C15" gate="G$1" pin="2"/>
+<wire x1="-48.26" y1="30.48" x2="-43.18" y2="30.48" width="0.1524" layer="91"/>
+<junction x="-48.26" y="30.48"/>
 </segment>
 <segment>
@@
 <junction x="-53.34" y="38.1"/>
 <label x="-63.5" y="43.18" size="1.778" layer="95"/>
+<pinref part="C15" gate="G$1" pin="1"/>
+<wire x1="-48.26" y1="38.1" x2="-43.18" y2="38.1" width="0.1524" layer="91"/>
+<junction x="-48.26" y="38.1"/>
 </segment>
 <segment>
@@
 </segment>
 <segment>
+<pinref part="IC1" gate="PORTB_H" pin="PB9"/>
+<wire x1="86.36" y1="66.04" x2="88.9" y2="66.04" width="0.1524" layer="91"/>
+<label x="88.9" y="66.04" size="1.778" layer="95"/>
+</segment>
+</net>
+<net name="PWM10" class="0">
+<segment>
+<pinref part="R10" gate="G$1" pin="2"/>
+<wire x1="25.4" y1="71.12" x2="27.94" y2="71.12" width="0.1524" layer="91"/>
+<label x="27.94" y="71.12" size="1.778" layer="95"/>
+</segment>
+<segment>
+<pinref part="IC1" gate="PORTB_H" pin="PB8"/>
+<wire x1="86.36" y1="68.58" x2="88.9" y2="68.58" width="0.1524" layer="91"/>
+<label x="88.9" y="68.58" size="1.778" layer="95"/>
+</segment>
+</net>
+<net name="PWM11" class="0">
+<segment>
+<pinref part="R11" gate="G$1" pin="2"/>
+<wire x1="25.4" y1="68.58" x2="27.94" y2="68.58" width="0.1524" layer="91"/>
+<label x="27.94" y="68.58" size="1.778" layer="95"/>
+</segment>
+<segment>
+<pinref part="IC1" gate="PORTB_L" pin="PB7"/>
+<wire x1="86.36" y1="76.2" x2="88.9" y2="76.2" width="0.1524" layer="91"/>
+<label x="88.9" y="76.2" size="1.778" layer="95"/>
+</segment>
+</net>
+<net name="PWM12" class="0">
+<segment>
+<pinref part="R12" gate="G$1" pin="2"/>
+<wire x1="25.4" y1="66.04" x2="27.94" y2="66.04" width="0.1524" layer="91"/>
+<label x="27.94" y="66.04" size="1.778" layer="95"/>
+</segment>
+<segment>
 <pinref part="IC1" gate="PORTB_L" pin="PB6"/>
 <wire x1="86.36" y1="78.74" x2="88.9" y2="78.74" width="0.1524" layer="91"/>
@@
 </segment>
 </net>
-<net name="PWM10" class="0">
-<segment>
-<pinref part="R10" gate="G$1" pin="2"/>
-<wire x1="25.4" y1="71.12" x2="27.94" y2="71.12" width="0.1524" layer="91"/>
-<label x="27.94" y="71.12" size="1.778" layer="95"/>
-</segment>
-<segment>
-<pinref part="IC1" gate="PORTB_L" pin="PB7"/>
-<wire x1="86.36" y1="76.2" x2="88.9" y2="76.2" width="0.1524" layer="91"/>
-<label x="88.9" y="76.2" size="1.778" layer="95"/>
-</segment>
-</net>
-<net name="PWM11" class="0">
-<segment>
-<pinref part="R11" gate="G$1" pin="2"/>
-<wire x1="25.4" y1="68.58" x2="27.94" y2="68.58" width="0.1524" layer="91"/>
-<label x="27.94" y="68.58" size="1.778" layer="95"/>
-</segment>
-<segment>
-<pinref part="IC1" gate="PORTB_H" pin="PB8"/>
-<wire x1="86.36" y1="68.58" x2="88.9" y2="68.58" width="0.1524" layer="91"/>
-<label x="88.9" y="68.58" size="1.778" layer="95"/>
-</segment>
-</net>
-<net name="PWM12" class="0">
-<segment>
-<pinref part="R12" gate="G$1" pin="2"/>
-<wire x1="25.4" y1="66.04" x2="27.94" y2="66.04" width="0.1524" layer="91"/>
-<label x="27.94" y="66.04" size="1.778" layer="95"/>
-</segment>
-<segment>
-<pinref part="IC1" gate="PORTB_H" pin="PB9"/>
-<wire x1="86.36" y1="66.04" x2="88.9" y2="66.04" width="0.1524" layer="91"/>
-<label x="88.9" y="66.04" size="1.778" layer="95"/>
-</segment>
-</net>
